File: WarBoard.kicad_sch (KiCad schematic)
At the start: 46 parts, among them J1 OLED_128x64, SW1 RotaryEncoder_Switch, SW2 RotaryEncoder_Switch, SW3 Reset, SW4 SW_SPDT_321, U1 WS2812B-4020, U10 DRV2505L, U3 SuperMini nRF52840, U4 WS2812B-4020, U5 WS2812B-4020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

Commit message: failsafe: checkpoint before battery wiring and net class fixes
Parts:
- added SW5: Switch, Button_Switch_SMD:SW_SPDT_Shouhan_MSK12C02, symbol ScottoKeebs:Placeholder_Switch
- SW4: footprint Button_Switch_SMD:SW_SPDT_CK_JS102011SAQN -> Button_Switch_THT:SW_Slide-03_Wuerth-WS-SLTV_10x2.5x6.4_P2.54mm
Connections:
- net at BT1.1 (+): now also SW5.1; no longer U3.29 (BAT+)
- new net: SW5.2, U3.29 (BAT+)
Other:
- moved on the sheet: BT1
Changed lines of the file:
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@@
 	(wire
 		(pts
+			(xy -591.82 67.31) (xy -589.28 67.31)
+		)
+		(stroke
+			(width 0)
+			(type default)
+		)
+	)
+	(wire
+		(pts
 			(xy -435.61 48.26) (xy -427.99 48.26)
 		)
@@
 	(wire
 		(pts
+			(xy -579.12 71.12) (xy -575.31 71.12)
+		)
+		(stroke
+			(width 0)
+			(type default)
+		)
+	)
+	(wire
+		(pts
 			(xy -461.01 73.66) (xy -448.31 73.66)
 		)
@@
 	(wire
 		(pts
-			(xy -613.41 74.93) (xy -595.63 74.93)
+			(xy -613.41 67.31) (xy -601.98 67.31)
 		)
 		(stroke
@@
 	(wire
 		(pts
-			(xy -613.41 74.93) (xy -613.41 81.28)
+			(xy -613.41 67.31) (xy -613.41 81.28)
 		)
 		(stroke
@@
 	(wire
 		(pts
-			(xy -585.47 74.93) (xy -575.31 74.93)
-		)
-		(stroke
-			(width 0)
-			(type default)
-		)
-	)
-	(wire
-		(pts
 			(xy -502.92 11.43) (xy -502.92 5.08)
 		)
@@
 	(wire
 		(pts
-			(xy -575.31 74.93) (xy -575.31 81.28)
+			(xy -445.77 177.8) (xy -415.29 177.8)
 		)
 		(stroke
@@
 	(wire
 		(pts
-			(xy -445.77 177.8) (xy -415.29 177.8)
+			(xy -453.39 34.29) (xy -453.39 38.1)
 		)
 		(stroke
@@
 	(wire
 		(pts
-			(xy -453.39 34.29) (xy -453.39 38.1)
+			(xy -478.79 50.8) (xy -478.79 63.5)
 		)
 		(stroke
@@
 	(wire
 		(pts
-			(xy -478.79 50.8) (xy -478.79 63.5)
+			(xy -461.01 60.96) (xy -448.31 60.96)
 		)
 		(stroke
@@
 	(wire
 		(pts
-			(xy -461.01 60.96) (xy -448.31 60.96)
+			(xy -466.09 50.8) (xy -466.09 63.5)
 		)
 		(stroke
@@
 	(wire
 		(pts
-			(xy -466.09 50.8) (xy -466.09 63.5)
+			(xy -589.28 67.31) (xy -589.28 71.12)
 		)
 		(stroke
@@
 	(wire
 		(pts
+			(xy -575.31 71.12) (xy -575.31 81.28)
+		)
+		(stroke
+			(width 0)
+			(type default)
+		)
+	)
+	(wire
+		(pts
 			(xy -360.68 114.3) (xy -360.68 110.49)
 		)
@@
 	(symbol
 		(lib_id "Device:Battery")
-		(at -590.55 74.93 270)
+		(at -596.9 67.31 270)
 		(unit 1)
 		(body_style 1)
@@
 		(dnp no)
 		(property "Reference" "BT1"
-			(at -590.55 70.104 90)
+			(at -596.9 62.484 90)
 			(show_name no)
 			(do_not_autoplace no)
@@
 		)
 		(property "Value" "3.7 V"
-			(at -590.55 71.882 90)
+			(at -596.9 64.262 90)
 			(show_name no)
 			(do_not_autoplace no)
@@
 		)
 		(property "Footprint" "ScottoKeebs_Scotto:Battery"
-			(at -589.026 74.93 90)
+			(at -595.376 67.31 90)
 			(hide yes)
 			(show_name no)
@@
 		)
 		(property "Datasheet" ""
-			(at -589.026 74.93 90)
+			(at -595.376 67.31 90)
 			(hide yes)
 			(show_name no)
@@
 		)
 		(property "Description" "Multiple-cell battery"
-			(at -590.55 74.93 0)
+			(at -596.9 67.31 0)
 			(hide yes)
 			(show_name no)
@@
 		)
 		(property "Sim.Device" "V"
-			(at -590.55 74.93 0)
+			(at -596.9 67.31 0)
 			(hide yes)
 			(show_name no)
@@
 		)
 		(property "Sim.Type" "DC"
-			(at -590.55 74.93 0)
+			(at -596.9 67.31 0)
 			(hide yes)
 			(show_name no)
@@
 		)
 		(property "Sim.Pins" "1=+ 2=-"
-			(at -590.55 74.93 0)
+			(at -596.9 67.31 0)
 			(hide yes)
 			(show_name no)
@@
 			)
 		)
-		(property "Footprint" "Button_Switch_SMD:SW_SPDT_CK_JS102011SAQN"
+		(property "Footprint" "Button_Switch_THT:SW_Slide-03_Wuerth-WS-SLTV_10x2.5x6.4_P2.54mm"
 			(at -590.55 139.7 0)
 			(hide yes)
@@
 					(unit 1)
 				)
+			)
+		)
+	)
+	(symbol
+		(lib_id "ScottoKeebs:Placeholder_Switch")
+		(at -584.2 71.12 0)
+		(unit 1)
+		(body_style 1)
+		(exclude_from_sim no)
+		(in_bom yes)
+		(on_board yes)
+		(in_pos_files yes)
+		(dnp no)
+		(fields_autoplaced yes)
+		(property "Reference" "SW5"
+			(at -584.2 63.5 0)
+			(show_name no)
+			(do_not_autoplace no)
+			(effects
+				(font
+					(size 1.27 1.27)
+				)
+			)
+		)
+		(property "Value" "Switch"
+			(at -584.2 66.04 0)
+			(show_name no)
+			(do_not_autoplace no)
+			(effects
+				(font
+					(size 1.27 1.27)
+				)
+			)
+		)
+		(property "Footprint" "Button_Switch_SMD:SW_SPDT_Shouhan_MSK12C02"
+			(at -584.2 66.04 0)
+			(hide yes)
+			(show_name no)
+			(do_not_autoplace no)
+			(effects
+				(font
+					(size 1.27 1.27)
+				)
+			)
+		)
+		(property "Datasheet" ""
+			(at -584.2 66.04 0)
+			(hide yes)
+			(show_name no)
+			(do_not_autoplace no)
+			(effects
+				(font
+					(size 1.27 1.27)
+				)
+			)
+		)
+		(property "Description" "Push button switch, generic, two pins"
+			(at -584.2 71.12 0)
+			(hide yes)
+			(show_name no)
+			(do_not_autoplace no)
+			(effects
+				(font
+					(size 1.27 1.27)
+				)
+			)
+		)
+		(pin "1"
+		)
+		(pin "2"
+		)
+		(instances
+			(project "WarBoard"
+				(path "/222a5836-0859-4d65-bff6-f9bdf97b6e3a"
+					(reference "SW5")
+					(unit 1)
+				)
