File: WarBoard.kicad_sch (KiCad schematic)
At the start: 47 parts, among them J1 OLED_128x64, SW1 RotaryEncoder_Switch, SW2 RotaryEncoder_Switch, SW3 Reset, SW4 SW_SPDT_321, SW5 Switch, U1 WS2812B-4020, U10 DRV2505L, U3 SuperMini nRF52840, U4 WS2812B-4020, U5 WS2812B-4020, U6 WS2812B-4020, U7 SKRHAAE010, U8 JoyStick, U9 MPU6050

Commit message: Final Iter
Connections:
- net JS: now reaches U8.5 (KEY)
- net JS: now also U3.12 (P1.06-LF)
- no-connect marks 13 -> 11
Changed lines of the file:
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@@
-	)
-	(no_connect
-		(at -613.41 111.76)
 	)
 	(no_connect
@@
 	)
 	(no_connect
-		(at -497.84 5.08)
-	)
-	(no_connect
 		(at -450.85 99.06)
 	)
@@
 		)
 	)
+	(global_label "JS"
+		(shape input)
+		(at -497.84 5.08 270)
+		(fields_autoplaced yes)
+		(effects
+			(font
+				(size 1.27 1.27)
+				(color 72 72 0 1)
+			)
+			(justify right)
+		)
+		(property "Intersheetrefs" "${INTERSHEET_REFS}"
+			(at -497.84 10.2423 90)
+			(hide yes)
+			(show_name no)
+			(do_not_autoplace no)
+			(effects
+				(font
+					(size 1.27 1.27)
+				)
+				(justify right)
+			)
+		)
+	)
 	(global_label "SW1_B"
 		(shape input)
@@
 			(hide yes)
 			(show_name no)
+			(do_not_autoplace no)
+			(effects
+				(font
+					(size 1.27 1.27)
+				)
+				(justify right)
+			)
+		)
+	)
+	(global_label "JS"
+		(shape input)
+		(at -613.41 111.76 180)
+		(fields_autoplaced yes)
+		(effects
+			(font
+				(size 1.27 1.27)
+				(color 72 72 0 1)
+			)
+			(justify right)
+		)
+		(property "Intersheetrefs" "${INTERSHEET_REFS}"
+			(at -618.5723 111.76 0)
+			(hide yes)
+			(show_name no)
